Commit message: added vrtp

File: drone_bringup/configuration_files/fixed_joint.urdf (robot description, URDF)
Before this commit: robot drone_fixed_joint, 3 links, 2 joints
Links:
- removed link t265_link
Joints:
- removed joint t265_joint_link
- joint d400_joint_link: origin xyz=0.12 0 0.0 rpy=0 0.0 0.0 -> xyz=0.9 0 -0.055 rpy=0 1.5708 0.0
